Commit message: Correct biped robot mass to measured 12.61 kg (was 11.34 kg / 10% light)
The real robot (legs + torso, no arms) weighs 27.8 lb = 12.61 kg, but the
CAD-derived biped asset totalled 11.34 kg (25.0 lb). Cross-checked against the
bench-measured assembled actuator weights (M6C12 680 g x8, MAD5010 425 g x4 =
7.14 kg, 57% of the robot): the sim's 12 leg links (8.18 kg) already carry that
motor mass correctly, so the entire 1.27 kg deficit is torso/structure (battery,
compute, wiring) missing from CAD.

Parked the deficit on the base/torso link: mass 3.16 -> 4.43 kg, diagonal +
product inertia scaled x1.4016 (added mass assumed distributed like the torso;
CoM kept). Applied as a root-layer override in usd/humanoid_biped.usd (what Isaac
loads) and mirrored in urdf/humanoid_biped.urdf. Full-humanoid asset and shared
physics config untouched. Total now 12.61 kg. See configs/actuators/PROVENANCE.md.

Co-Authored-By: Claude Opus 4.8 (1M context) <noreply@anthropic.com>

File: source/humanoid_policy_assets/data/robots/humanoid/urdf/humanoid_biped.urdf (robot description, URDF)
Before this commit: robot humanoid, 15 links, 14 joints
Links:
- link base: mass 3.16059 -> 4.42983
